Commit message: Tweaked the sim

File: ROS/catkin_ws/src/Sim_description/urdf/Sim.xacro (robot description, xacro)
@@ -6,5 +6,5 @@
 <link name="base_link">
   <inertial>
-    <origin rpy="0 0 0" xyz="0.0006007577009604423 0.0 0.07512755869305572"/>
+    <origin rpy="0 0 0" xyz="0.0006007577009604456 -2.0009250954814774e-19 0.1912775586930594"/>
     <mass value="105.11118623932714"/>
     <inertia ixx="3.347522" ixy="0.0" ixz="-0.005562" iyy="10.805776" iyz="0.0" izz="13.757255"/>
@@ -26,10 +26,10 @@
 <link name="wheel1_1">
   <inertial>
-    <origin rpy="0 0 0" xyz="4.551914400963142e-15 -0.03311871322111437 1.3877787807814457e-17"/>
+    <origin rpy="0 0 0" xyz="4.440892098500626e-15 -0.033118713221114426 -0.11614999999999634"/>
     <mass value="5.16787815760831"/>
     <inertia ixx="0.032523" ixy="0.0" ixz="0.0" iyy="0.060048" iyz="0.0" izz="0.032523"/>
   </inertial>
   <visual>
-    <origin rpy="0 0 0" xyz="-0.275 0.31 -0.03625"/>
+    <origin rpy="0 0 0" xyz="-0.275 0.31 -0.26855"/>
     <geometry>
       <mesh filename="package://Sim_description/meshes/wheel1_1.stl" scale="0.001 0.001 0.001"/>
@@ -38,5 +38,5 @@
   </visual>
   <collision>
-    <origin rpy="0 0 0" xyz="-0.275 0.31 -0.03625"/>
+    <origin rpy="0 0 0" xyz="-0.275 0.31 -0.26855"/>
     <geometry>
       <mesh filename="package://Sim_description/meshes/wheel1_1.stl" scale="0.001 0.001 0.001"/>
@@ -46,10 +46,10 @@
 <link name="wheel4_1">
   <inertial>
-    <origin rpy="0 0 0" xyz="-4.440892098500626e-15 -0.03311871322111437 1.3877787807814457e-17"/>
+    <origin rpy="0 0 0" xyz="-4.6074255521944e-15 -0.033118713221114315 -0.11614999999999634"/>
     <mass value="5.16787815760831"/>
-    <inertia ixx="0.032523" ixy="-0.0" ixz="0.0" iyy="0.060048" iyz="0.0" izz="0.032523"/>
+    <inertia ixx="0.032523" ixy="0.0" ixz="0.0" iyy="0.060048" iyz="-0.0" izz="0.032523"/>
   </inertial>
   <visual>
-    <origin rpy="0 0 0" xyz="0.275 0.31 -0.03625"/>
+    <origin rpy="0 0 0" xyz="0.275 0.31 -0.26855"/>
     <geometry>
       <mesh filename="package://Sim_description/meshes/wheel4_1.stl" scale="0.001 0.001 0.001"/>
@@ -58,5 +58,5 @@
   </visual>
   <collision>
-    <origin rpy="0 0 0" xyz="0.275 0.31 -0.03625"/>
+    <origin rpy="0 0 0" xyz="0.275 0.31 -0.26855"/>
     <geometry>
       <mesh filename="package://Sim_description/meshes/wheel4_1.stl" scale="0.001 0.001 0.001"/>
@@ -66,10 +66,10 @@
 <link name="wheel2_1">
   <inertial>
-    <origin rpy="0 0 0" xyz="0.0 0.03311871322111437 1.3877787807814457e-17"/>
+    <origin rpy="0 0 0" xyz="1.1102230246251565e-16 0.033118713221114315 -0.11614999999999634"/>
     <mass value="5.16787815760831"/>
-    <inertia ixx="0.032523" ixy="0.0" ixz="0.0" iyy="0.060048" iyz="-0.0" izz="0.032523"/>
+    <inertia ixx="0.032523" ixy="0.0" ixz="0.0" iyy="0.060048" iyz="0.0" izz="0.032523"/>
   </inertial>
   <visual>
-    <origin rpy="0 0 0" xyz="-0.275 -0.31 -0.03625"/>
+    <origin rpy="0 0 0" xyz="-0.275 -0.31 -0.26855"/>
     <geometry>
       <mesh filename="package://Sim_description/meshes/wheel2_1.stl" scale="0.001 0.001 0.001"/>
@@ -78,5 +78,5 @@
   </visual>
   <collision>
-    <origin rpy="0 0 0" xyz="-0.275 -0.31 -0.03625"/>
+    <origin rpy="0 0 0" xyz="-0.275 -0.31 -0.26855"/>
     <geometry>
       <mesh filename="package://Sim_description/meshes/wheel2_1.stl" scale="0.001 0.001 0.001"/>
@@ -86,10 +86,10 @@
 <link name="wheel3_1">
   <inertial>
-    <origin rpy="0 0 0" xyz="0.0 0.03311871322111437 1.3877787807814457e-17"/>
+    <origin rpy="0 0 0" xyz="1.6653345369377348e-16 0.033118713221114426 -0.11614999999999634"/>
     <mass value="5.16787815760831"/>
     <inertia ixx="0.032523" ixy="0.0" ixz="0.0" iyy="0.060048" iyz="-0.0" izz="0.032523"/>
   </inertial>
   <visual>
-    <origin rpy="0 0 0" xyz="0.275 -0.31 -0.03625"/>
+    <origin rpy="0 0 0" xyz="0.275 -0.31 -0.26855"/>
     <geometry>
       <mesh filename="package://Sim_description/meshes/wheel3_1.stl" scale="0.001 0.001 0.001"/>
@@ -98,5 +98,5 @@
   </visual>
   <collision>
-    <origin rpy="0 0 0" xyz="0.275 -0.31 -0.03625"/>
+    <origin rpy="0 0 0" xyz="0.275 -0.31 -0.26855"/>
     <geometry>
       <mesh filename="package://Sim_description/meshes/wheel3_1.stl" scale="0.001 0.001 0.001"/>
@@ -106,10 +106,10 @@
 <link name="lidar_1">
   <inertial>
-    <origin rpy="0 0 0" xyz="5.551115123125783e-17 -5.5845130209510275e-18 0.012500000000000011"/>
+    <origin rpy="0 0 0" xyz="5.551115123125783e-17 -1.388112759759698e-16 0.01250000000000362"/>
     <mass value="0.10789485809488791"/>
-    <inertia ixx="4.1e-05" ixy="0.0" ixz="0.0" iyy="4.1e-05" iyz="-0.0" izz="7e-05"/>
+    <inertia ixx="4.1e-05" ixy="-0.0" ixz="0.0" iyy="4.1e-05" iyz="-0.0" izz="7e-05"/>
   </inertial>
   <visual>
-    <origin rpy="0 0 0" xyz="-0.4 -0.0 -0.18"/>
+    <origin rpy="0 0 0" xyz="-0.4 0.0 -0.29615"/>
     <geometry>
       <mesh filename="package://Sim_description/meshes/lidar_1.stl" scale="0.001 0.001 0.001"/>
@@ -118,5 +118,5 @@
   </visual>
   <collision>
-    <origin rpy="0 0 0" xyz="-0.4 -0.0 -0.18"/>
+    <origin rpy="0 0 0" xyz="-0.4 0.0 -0.29615"/>
     <geometry>
       <mesh filename="package://Sim_description/meshes/lidar_1.stl" scale="0.001 0.001 0.001"/>
@@ -125,17 +125,17 @@
 </link>
 <joint name="Rev1" type="continuous">
-  <origin rpy="0 0 0" xyz="0.275 -0.31 0.03625"/>
+  <origin rpy="0 0 0" xyz="0.275 -0.31 0.26855"/>
   <parent link="base_link"/>
   <child link="wheel1_1"/>
-  <axis xyz="0.0 -1.0 0.0"/>
+  <axis xyz="-0.0 -1.0 0.0"/>
 </joint>
 <joint name="Rev2" type="continuous">
-  <origin rpy="0 0 0" xyz="-0.275 -0.31 0.03625"/>
+  <origin rpy="0 0 0" xyz="-0.275 -0.31 0.26855"/>
   <parent link="base_link"/>
   <child link="wheel4_1"/>
-  <axis xyz="0.0 -1.0 0.0"/>
+  <axis xyz="-0.0 -1.0 0.0"/>
 </joint>
 <joint name="Rev3" type="continuous">
-  <origin rpy="0 0 0" xyz="0.275 0.31 0.03625"/>
+  <origin rpy="0 0 0" xyz="0.275 0.31 0.26855"/>
   <parent link="base_link"/>
   <child link="wheel2_1"/>
@@ -143,5 +143,5 @@
 </joint>
 <joint name="Rev4" type="continuous">
-  <origin rpy="0 0 0" xyz="-0.275 0.31 0.03625"/>
+  <origin rpy="0 0 0" xyz="-0.275 0.31 0.26855"/>
   <parent link="base_link"/>
   <child link="wheel3_1"/>
@@ -149,5 +149,5 @@
 </joint>
 <joint name="Rigid5" type="fixed">
-  <origin rpy="0 0 0" xyz="0.4 0.0 0.18"/>
+  <origin rpy="0 0 0" xyz="0.4 0.0 0.29615"/>
   <parent link="base_link"/>
   <child link="lidar_1"/>

Commit message: Sim Testing

File: ROS/catkin_ws/src/Sim_description/urdf/Sim.xacro (robot description, xacro)
@@ -26,10 +26,10 @@
 <link name="wheel1_1">
   <inertial>
-    <origin rpy="0 0 0" xyz="4.440892098500626e-15 -0.033118713221114426 -0.11614999999999634"/>
-    <mass value="5.16787815760831"/>
-    <inertia ixx="0.032523" ixy="0.0" ixz="0.0" iyy="0.060048" iyz="0.0" izz="0.032523"/>
+    <origin rpy="0 0 0" xyz="-1.1102230246251565e-16 -0.03810000000000002 3.6914915568786455e-15"/>
+    <mass value="5.17079983877615"/>
+    <inertia ixx="0.032526" ixy="0.0" ixz="0.0" iyy="0.060048" iyz="0.0" izz="0.032526"/>
   </inertial>
   <visual>
-    <origin rpy="0 0 0" xyz="-0.275 0.31 -0.26855"/>
+    <origin rpy="0 0 0" xyz="-0.275 0.31 -0.1524"/>
     <geometry>
       <mesh filename="package://Sim_description/meshes/wheel1_1.stl" scale="0.001 0.001 0.001"/>
@@ -38,5 +38,5 @@
   </visual>
   <collision>
-    <origin rpy="0 0 0" xyz="-0.275 0.31 -0.26855"/>
+    <origin rpy="0 0 0" xyz="-0.275 0.31 -0.1524"/>
     <geometry>
       <mesh filename="package://Sim_description/meshes/wheel1_1.stl" scale="0.001 0.001 0.001"/>
@@ -46,10 +46,10 @@
 <link name="wheel4_1">
   <inertial>
-    <origin rpy="0 0 0" xyz="-4.6074255521944e-15 -0.033118713221114315 -0.11614999999999634"/>
-    <mass value="5.16787815760831"/>
-    <inertia ixx="0.032523" ixy="0.0" ixz="0.0" iyy="0.060048" iyz="-0.0" izz="0.032523"/>
+    <origin rpy="0 0 0" xyz="-5.551115123125783e-17 -0.038099999999999856 3.6914915568786455e-15"/>
+    <mass value="5.17079983877615"/>
+    <inertia ixx="0.032526" ixy="-0.0" ixz="0.0" iyy="0.060048" iyz="0.0" izz="0.032526"/>
   </inertial>
   <visual>
-    <origin rpy="0 0 0" xyz="0.275 0.31 -0.26855"/>
+    <origin rpy="0 0 0" xyz="0.275 0.31 -0.1524"/>
     <geometry>
       <mesh filename="package://Sim_description/meshes/wheel4_1.stl" scale="0.001 0.001 0.001"/>
@@ -58,5 +58,5 @@
   </visual>
   <collision>
-    <origin rpy="0 0 0" xyz="0.275 0.31 -0.26855"/>
+    <origin rpy="0 0 0" xyz="0.275 0.31 -0.1524"/>
     <geometry>
       <mesh filename="package://Sim_description/meshes/wheel4_1.stl" scale="0.001 0.001 0.001"/>
@@ -64,12 +64,32 @@
   </collision>
 </link>
+<link name="wheel3_1">
+  <inertial>
+    <origin rpy="0 0 0" xyz="1.1102230246251565e-16 0.03810000000000002 3.6914915568786455e-15"/>
+    <mass value="5.17079983877615"/>
+    <inertia ixx="0.032526" ixy="-0.0" ixz="0.0" iyy="0.060048" iyz="-0.0" izz="0.032526"/>
+  </inertial>
+  <visual>
+    <origin rpy="0 0 0" xyz="0.275 -0.31 -0.1524"/>
+    <geometry>
+      <mesh filename="package://Sim_description/meshes/wheel3_1.stl" scale="0.001 0.001 0.001"/>
+    </geometry>
+    <material name="silver"/>
+  </visual>
+  <collision>
+    <origin rpy="0 0 0" xyz="0.275 -0.31 -0.1524"/>
+    <geometry>
+      <mesh filename="package://Sim_description/meshes/wheel3_1.stl" scale="0.001 0.001 0.001"/>
+    </geometry>
+  </collision>
+</link>
 <link name="wheel2_1">
   <inertial>
-    <origin rpy="0 0 0" xyz="1.1102230246251565e-16 0.033118713221114315 -0.11614999999999634"/>
-    <mass value="5.16787815760831"/>
-    <inertia ixx="0.032523" ixy="0.0" ixz="0.0" iyy="0.060048" iyz="0.0" izz="0.032523"/>
+    <origin rpy="0 0 0" xyz="1.1102230246251565e-16 0.038099999999999856 3.6914915568786455e-15"/>
+    <mass value="5.17079983877615"/>
+    <inertia ixx="0.032526" ixy="0.0" ixz="0.0" iyy="0.060048" iyz="0.0" izz="0.032526"/>
   </inertial>
   <visual>
-    <origin rpy="0 0 0" xyz="-0.275 -0.31 -0.26855"/>
+    <origin rpy="0 0 0" xyz="-0.275 -0.31 -0.1524"/>
     <geometry>
       <mesh filename="package://Sim_description/meshes/wheel2_1.stl" scale="0.001 0.001 0.001"/>
@@ -78,5 +98,5 @@
   </visual>
   <collision>
-    <origin rpy="0 0 0" xyz="-0.275 -0.31 -0.26855"/>
+    <origin rpy="0 0 0" xyz="-0.275 -0.31 -0.1524"/>
     <geometry>
       <mesh filename="package://Sim_description/meshes/wheel2_1.stl" scale="0.001 0.001 0.001"/>
@@ -84,72 +104,27 @@
   </collision>
 </link>
-<link name="wheel3_1">
-  <inertial>
-    <origin rpy="0 0 0" xyz="1.6653345369377348e-16 0.033118713221114426 -0.11614999999999634"/>
-    <mass value="5.16787815760831"/>
-    <inertia ixx="0.032523" ixy="0.0" ixz="0.0" iyy="0.060048" iyz="-0.0" izz="0.032523"/>
-  </inertial>
-  <visual>
-    <origin rpy="0 0 0" xyz="0.275 -0.31 -0.26855"/>
-    <geometry>
-      <mesh filename="package://Sim_description/meshes/wheel3_1.stl" scale="0.001 0.001 0.001"/>
-    </geometry>
-    <material name="silver"/>
-  </visual>
-  <collision>
-    <origin rpy="0 0 0" xyz="0.275 -0.31 -0.26855"/>
-    <geometry>
-      <mesh filename="package://Sim_description/meshes/wheel3_1.stl" scale="0.001 0.001 0.001"/>
-    </geometry>
-  </collision>
-</link>
-<link name="lidar_1">
-  <inertial>
-    <origin rpy="0 0 0" xyz="5.551115123125783e-17 -1.388112759759698e-16 0.01250000000000362"/>
-    <mass value="0.10789485809488791"/>
-    <inertia ixx="4.1e-05" ixy="-0.0" ixz="0.0" iyy="4.1e-05" iyz="-0.0" izz="7e-05"/>
-  </inertial>
-  <visual>
-    <origin rpy="0 0 0" xyz="-0.4 0.0 -0.29615"/>
-    <geometry>
-      <mesh filename="package://Sim_description/meshes/lidar_1.stl" scale="0.001 0.001 0.001"/>
-    </geometry>
-    <material name="silver"/>
-  </visual>
-  <collision>
-    <origin rpy="0 0 0" xyz="-0.4 0.0 -0.29615"/>
-    <geometry>
-      <mesh filename="package://Sim_description/meshes/lidar_1.stl" scale="0.001 0.001 0.001"/>
-    </geometry>
-  </collision>
-</link>
-<joint name="Rev1" type="continuous">
-  <origin rpy="0 0 0" xyz="0.275 -0.31 0.26855"/>
+<joint name="Rev6" type="continuous">
+  <origin rpy="0 0 0" xyz="0.275 -0.31 0.1524"/>
   <parent link="base_link"/>
   <child link="wheel1_1"/>
   <axis xyz="-0.0 -1.0 0.0"/>
 </joint>
-<joint name="Rev2" type="continuous">
-  <origin rpy="0 0 0" xyz="-0.275 -0.31 0.26855"/>
+<joint name="Rev7" type="continuous">
+  <origin rpy="0 0 0" xyz="-0.275 -0.31 0.1524"/>
   <parent link="base_link"/>
   <child link="wheel4_1"/>
   <axis xyz="-0.0 -1.0 0.0"/>
 </joint>
-<joint name="Rev3" type="continuous">
-  <origin rpy="0 0 0" xyz="0.275 0.31 0.26855"/>
+<joint name="Rev8" type="continuous">
+  <origin rpy="0 0 0" xyz="-0.275 0.31 0.1524"/>
+  <parent link="base_link"/>
+  <child link="wheel3_1"/>
+  <axis xyz="0.0 1.0 0.0"/>
+</joint>
+<joint name="Rev9" type="continuous">
+  <origin rpy="0 0 0" xyz="0.275 0.31 0.1524"/>
   <parent link="base_link"/>
   <child link="wheel2_1"/>
   <axis xyz="0.0 1.0 0.0"/>
 </joint>
-<joint name="Rev4" type="continuous">
-  <origin rpy="0 0 0" xyz="-0.275 0.31 0.26855"/>
-  <parent link="base_link"/>
-  <child link="wheel3_1"/>
-  <axis xyz="0.0 1.0 0.0"/>
-</joint>
-<joint name="Rigid5" type="fixed">
-  <origin rpy="0 0 0" xyz="0.4 0.0 0.29615"/>
-  <parent link="base_link"/>
-  <child link="lidar_1"/>
-</joint>
 </robot>

Commit message: More Sim Tweaking

File: ROS/catkin_ws/src/Sim_description/urdf/Sim.xacro (robot description, xacro)
@@ -104,4 +104,24 @@
   </collision>
 </link>
+<link name="lidar_1">
+  <inertial>
+    <origin rpy="0 0 0" xyz="5.551115123125783e-17 -1.388112759759698e-16 0.01250000000000362"/>
+    <mass value="0.10789485809488791"/>
+    <inertia ixx="4.1e-05" ixy="-0.0" ixz="0.0" iyy="4.1e-05" iyz="-0.0" izz="7e-05"/>
+  </inertial>
+  <visual>
+    <origin rpy="0 0 0" xyz="-0.4 0.0 -0.29615"/>
+    <geometry>
+      <mesh filename="package://Sim_description/meshes/lidar_1.stl" scale="0.001 0.001 0.001"/>
+    </geometry>
+    <material name="silver"/>
+  </visual>
+  <collision>
+    <origin rpy="0 0 0" xyz="-0.4 0.0 -0.29615"/>
+    <geometry>
+      <mesh filename="package://Sim_description/meshes/lidar_1.stl" scale="0.001 0.001 0.001"/>
+    </geometry>
+  </collision>
+</link>
 <joint name="Rev6" type="continuous">
   <origin rpy="0 0 0" xyz="0.275 -0.31 0.1524"/>
@@ -128,3 +148,8 @@
   <axis xyz="0.0 1.0 0.0"/>
 </joint>
+<joint name="Rigid10" type="fixed">
+  <origin rpy="0 0 0" xyz="0.4 0.0 0.29615"/>
+  <parent link="base_link"/>
+  <child link="lidar_1"/>
+</joint>
 </robot>
