Commit message: ROS new model

File: Modules/ROS/catkin_ws/src/rover_sim/urdf/Sim.xacro (robot description, xacro)
@@ -6,10 +6,10 @@
 <link name="base_link">
   <inertial>
-    <origin rpy="0 0 0" xyz="0.0006007577009604456 -2.0009250954814774e-19 0.1912775586930594"/>
-    <mass value="105.11118623932714"/>
-    <inertia ixx="3.347522" ixy="0.0" ixz="-0.005562" iyy="10.805776" iyz="0.0" izz="13.757255"/>
+    <origin xyz="-0.010217176975484165 2.035332124121442e-16 0.15794635989902708" rpy="0 0 0"/>
+    <mass value="43.16198403094287"/>
+    <inertia ixx="0.686298" iyy="4.62213" izz="5.125629" ixy="0.0" iyz="0.0" ixz="0.111555"/>
   </inertial>
   <visual>
-    <origin rpy="0 0 0" xyz="0 0 0"/>
+    <origin xyz="0 0 0" rpy="0 0 0"/>
     <geometry>
       <mesh filename="package://rover_sim/meshes/base_link.stl" scale="0.001 0.001 0.001"/>
@@ -18,5 +18,5 @@
   </visual>
   <collision>
-    <origin rpy="0 0 0" xyz="0 0 0"/>
+    <origin xyz="0 0 0" rpy="0 0 0"/>
     <geometry>
       <mesh filename="package://rover_sim/meshes/base_link.stl" scale="0.001 0.001 0.001"/>
@@ -24,12 +24,52 @@
   </collision>
 </link>
+<link name="wheel3_1">
+  <inertial>
+    <origin xyz="1.1102230246251565e-16 0.03810000000000002 3.6914915568786455e-15" rpy="0 0 0"/>
+    <mass value="5.17079983877615"/>
+    <inertia ixx="0.032526" iyy="0.060048" izz="0.032526" ixy="0.0" iyz="-0.0" ixz="0.0"/>
+  </inertial>
+  <visual>
+    <origin xyz="0.275 -0.21 -0.1524" rpy="0 0 0"/>
+    <geometry>
+      <mesh filename="package://rover_sim/meshes/wheel3_1.stl" scale="0.001 0.001 0.001"/>
+    </geometry>
+    <material name="silver"/>
+  </visual>
+  <collision>
+    <origin xyz="0.275 -0.21 -0.1524" rpy="0 0 0"/>
+    <geometry>
+      <mesh filename="package://rover_sim/meshes/wheel3_1.stl" scale="0.001 0.001 0.001"/>
+    </geometry>
+  </collision>
+</link>
+<link name="wheel2_1">
+  <inertial>
+    <origin xyz="5.551115123125783e-17 0.038099999999999884 3.6914915568786455e-15" rpy="0 0 0"/>
+    <mass value="5.17079983877615"/>
+    <inertia ixx="0.032526" iyy="0.060048" izz="0.032526" ixy="0.0" iyz="0.0" ixz="0.0"/>
+  </inertial>
+  <visual>
+    <origin xyz="-0.275 -0.21 -0.1524" rpy="0 0 0"/>
+    <geometry>
+      <mesh filename="package://rover_sim/meshes/wheel2_1.stl" scale="0.001 0.001 0.001"/>
+    </geometry>
+    <material name="silver"/>
+  </visual>
+  <collision>
+    <origin xyz="-0.275 -0.21 -0.1524" rpy="0 0 0"/>
+    <geometry>
+      <mesh filename="package://rover_sim/meshes/wheel2_1.stl" scale="0.001 0.001 0.001"/>
+    </geometry>
+  </collision>
+</link>
 <link name="wheel1_1">
   <inertial>
-    <origin rpy="0 0 0" xyz="-1.1102230246251565e-16 -0.03810000000000002 3.6914915568786455e-15"/>
+    <origin xyz="-5.551115123125783e-17 -0.03810000000000002 3.6914915568786455e-15" rpy="0 0 0"/>
     <mass value="5.17079983877615"/>
-    <inertia ixx="0.032526" ixy="0.0" ixz="0.0" iyy="0.060048" iyz="0.0" izz="0.032526"/>
+    <inertia ixx="0.032526" iyy="0.060048" izz="0.032526" ixy="0.0" iyz="0.0" ixz="0.0"/>
   </inertial>
   <visual>
-    <origin rpy="0 0 0" xyz="-0.275 0.31 -0.1524"/>
+    <origin xyz="-0.275 0.21 -0.1524" rpy="0 0 0"/>
     <geometry>
       <mesh filename="package://rover_sim/meshes/wheel1_1.stl" scale="0.001 0.001 0.001"/>
@@ -38,5 +78,5 @@
   </visual>
   <collision>
-    <origin rpy="0 0 0" xyz="-0.275 0.31 -0.1524"/>
+    <origin xyz="-0.275 0.21 -0.1524" rpy="0 0 0"/>
     <geometry>
       <mesh filename="package://rover_sim/meshes/wheel1_1.stl" scale="0.001 0.001 0.001"/>
@@ -46,10 +86,10 @@
 <link name="wheel4_1">
   <inertial>
-    <origin rpy="0 0 0" xyz="-5.551115123125783e-17 -0.038099999999999856 3.6914915568786455e-15"/>
+    <origin xyz="-5.551115123125783e-17 -0.038099999999999884 3.6914915568786455e-15" rpy="0 0 0"/>
     <mass value="5.17079983877615"/>
-    <inertia ixx="0.032526" ixy="-0.0" ixz="0.0" iyy="0.060048" iyz="0.0" izz="0.032526"/>
+    <inertia ixx="0.032526" iyy="0.060048" izz="0.032526" ixy="0.0" iyz="-0.0" ixz="-0.0"/>
   </inertial>
   <visual>
-    <origin rpy="0 0 0" xyz="0.275 0.31 -0.1524"/>
+    <origin xyz="0.275 0.21 -0.1524" rpy="0 0 0"/>
     <geometry>
       <mesh filename="package://rover_sim/meshes/wheel4_1.stl" scale="0.001 0.001 0.001"/>
@@ -58,5 +98,5 @@
   </visual>
   <collision>
-    <origin rpy="0 0 0" xyz="0.275 0.31 -0.1524"/>
+    <origin xyz="0.275 0.21 -0.1524" rpy="0 0 0"/>
     <geometry>
       <mesh filename="package://rover_sim/meshes/wheel4_1.stl" scale="0.001 0.001 0.001"/>
@@ -64,41 +104,21 @@
   </collision>
 </link>
-<link name="wheel3_1">
+<link name="dump_1">
   <inertial>
-    <origin rpy="0 0 0" xyz="1.1102230246251565e-16 0.03810000000000002 3.6914915568786455e-15"/>
-    <mass value="5.17079983877615"/>
-    <inertia ixx="0.032526" ixy="-0.0" ixz="0.0" iyy="0.060048" iyz="-0.0" izz="0.032526"/>
+    <origin xyz="0.17003553115914338 0.17922499310589943 -0.20554520775582574" rpy="0 0 0"/>
+    <mass value="65.04406534684018"/>
+    <inertia ixx="1.921537" iyy="2.093764" izz="2.246735" ixy="0.000408" iyz="-0.043648" ixz="-0.000475"/>
   </inertial>
   <visual>
-    <origin rpy="0 0 0" xyz="0.275 -0.31 -0.1524"/>
+    <origin xyz="0.525 0.165 -0.54615" rpy="0 0 0"/>
     <geometry>
-      <mesh filename="package://rover_sim/meshes/wheel3_1.stl" scale="0.001 0.001 0.001"/>
+      <mesh filename="package://rover_sim/meshes/dump_1.stl" scale="0.001 0.001 0.001"/>
     </geometry>
     <material name="silver"/>
   </visual>
   <collision>
-    <origin rpy="0 0 0" xyz="0.275 -0.31 -0.1524"/>
+    <origin xyz="0.525 0.165 -0.54615" rpy="0 0 0"/>
     <geometry>
-      <mesh filename="package://rover_sim/meshes/wheel3_1.stl" scale="0.001 0.001 0.001"/>
-    </geometry>
-  </collision>
-</link>
-<link name="wheel2_1">
-  <inertial>
-    <origin rpy="0 0 0" xyz="1.1102230246251565e-16 0.038099999999999856 3.6914915568786455e-15"/>
-    <mass value="5.17079983877615"/>
-    <inertia ixx="0.032526" ixy="0.0" ixz="0.0" iyy="0.060048" iyz="0.0" izz="0.032526"/>
-  </inertial>
-  <visual>
-    <origin rpy="0 0 0" xyz="-0.275 -0.31 -0.1524"/>
-    <geometry>
-      <mesh filename="package://rover_sim/meshes/wheel2_1.stl" scale="0.001 0.001 0.001"/>
-    </geometry>
-    <material name="silver"/>
-  </visual>
-  <collision>
-    <origin rpy="0 0 0" xyz="-0.275 -0.31 -0.1524"/>
-    <geometry>
-      <mesh filename="package://rover_sim/meshes/wheel2_1.stl" scale="0.001 0.001 0.001"/>
+      <mesh filename="package://rover_sim/meshes/dump_1.stl" scale="0.001 0.001 0.001"/>
     </geometry>
   </collision>
@@ -106,10 +126,10 @@
 <link name="lidar_1">
   <inertial>
-    <origin rpy="0 0 0" xyz="5.551115123125783e-17 -1.388112759759698e-16 0.01250000000000362"/>
+    <origin xyz="1.6653345369377348e-16 -1.3322676295501885e-16 0.012500000000003703" rpy="0 0 0"/>
     <mass value="0.10789485809488791"/>
-    <inertia ixx="4.1e-05" ixy="-0.0" ixz="0.0" iyy="4.1e-05" iyz="-0.0" izz="7e-05"/>
+    <inertia ixx="4.1e-05" iyy="4.1e-05" izz="7e-05" ixy="0.0" iyz="-0.0" ixz="0.0"/>
   </inertial>
   <visual>
-    <origin rpy="0 0 0" xyz="-0.4 0.0 -0.29615"/>
+    <origin xyz="-0.4 0.0 -0.24115" rpy="0 0 0"/>
     <geometry>
       <mesh filename="package://rover_sim/meshes/lidar_1.stl" scale="0.001 0.001 0.001"/>
@@ -118,5 +138,5 @@
   </visual>
   <collision>
-    <origin rpy="0 0 0" xyz="-0.4 0.0 -0.29615"/>
+    <origin xyz="-0.4 0.0 -0.24115" rpy="0 0 0"/>
     <geometry>
       <mesh filename="package://rover_sim/meshes/lidar_1.stl" scale="0.001 0.001 0.001"/>
@@ -124,32 +144,36 @@
   </collision>
 </link>
-<joint name="Rev6" type="continuous">
-  <origin rpy="0 0 0" xyz="0.275 -0.31 0.1524"/>
-  <parent link="base_link"/>
-  <child link="wheel1_1"/>
-  <axis xyz="-0.0 1.0 0.0"/>
-  <!--  xyz="-0.0 -1.0 0.0" -->
-</joint>
-<joint name="Rev7" type="continuous">
-  <origin rpy="0 0 0" xyz="-0.275 -0.31 0.1524"/>
-  <parent link="base_link"/>
-  <child link="wheel4_1"/>
-  <axis xyz="-0.0 1.0 0.0"/>
-  <!--  xyz="-0.0 -1.0 0.0" -->
-</joint>
-<joint name="Rev8" type="continuous">
-  <origin rpy="0 0 0" xyz="-0.275 0.31 0.1524"/>
+<joint name="Rev13" type="continuous">
+  <origin xyz="-0.275 0.21 0.1524" rpy="0 0 0"/>
   <parent link="base_link"/>
   <child link="wheel3_1"/>
   <axis xyz="0.0 1.0 0.0"/>
 </joint>
-<joint name="Rev9" type="continuous">
-  <origin rpy="0 0 0" xyz="0.275 0.31 0.1524"/>
+<joint name="Rev14" type="continuous">
+  <origin xyz="0.275 0.21 0.1524" rpy="0 0 0"/>
   <parent link="base_link"/>
   <child link="wheel2_1"/>
   <axis xyz="0.0 1.0 0.0"/>
 </joint>
-<joint name="Rigid10" type="fixed">
-  <origin rpy="0 0 0" xyz="0.4 0.0 0.29615"/>
+<joint name="Rev15" type="continuous">
+  <origin xyz="0.275 -0.21 0.1524" rpy="0 0 0"/>
+  <parent link="base_link"/>
+  <child link="wheel1_1"/>
+  <axis xyz="-0.0 -1.0 0.0"/>
+</joint>
+<joint name="Rev16" type="continuous">
+  <origin xyz="-0.275 -0.21 0.1524" rpy="0 0 0"/>
+  <parent link="base_link"/>
+  <child link="wheel4_1"/>
+  <axis xyz="0.0 1.0 0.0"/>
+</joint>
+<joint name="Rev17" type="fixed">
+  <origin xyz="-0.525 -0.165 0.54615" rpy="0 0 0"/>
+  <parent link="base_link"/>
+  <child link="dump_1"/>
+  <axis xyz="0.0 1.0 0.0"/>
+</joint>
+<joint name="Rigid18" type="fixed">
+  <origin xyz="0.4 0.0 0.24115" rpy="0 0 0"/>
   <parent link="base_link"/>
   <child link="lidar_1"/>
